Commit message: vito with left and right hands

File: vito_description/robots/vito.urdf.xacro (robot description, xacro)
@@ -28,9 +28,9 @@
       rpy="${M_PI*-40.8933907/180} ${M_PI*48.5903708/180} ${M_PI*40.8933907/180}"/>
   </xacro:kuka_lwr>
-  <xacro:soft_hand parent="left_arm_7_link" name="left_hand" withAdaptiveTransmission="true" useMimicTag="$(arg use_mimic_tag)">
-    <origin xyz="0 0 0" rpy="1.570796 0 0"/>
+  <xacro:soft_hand parent="left_arm_7_link" name="left_hand" left="true" withAdaptiveTransmission="true" useMimicTag="$(arg use_mimic_tag)">
+    <origin xyz="0 0 0" rpy="0 0 0"/>
   </xacro:soft_hand>
-  <xacro:soft_hand parent="right_arm_7_link" name="right_hand" withAdaptiveTransmission="true" useMimicTag="$(arg use_mimic_tag)">
-    <origin xyz="0 0 0" rpy="1.570796 0 0"/>
+  <xacro:soft_hand parent="right_arm_7_link" name="right_hand" left="false" withAdaptiveTransmission="true" useMimicTag="$(arg use_mimic_tag)">
+    <origin xyz="0 0 0" rpy="0 0 0"/>
   </xacro:soft_hand>
   <xacro:kit_head name="head" parent="world">
