Commit message: vito update: added hands and kit head

File: vito_description/model/table.urdf.xacro (robot description, xacro)
@@ -26,5 +26,5 @@
     <joint name="${parent}_${name}_base_joint" type="fixed">
         <insert_block name="origin"/>
-        <parent link="${parent}_link"/>
+        <parent link="${parent}"/>
         <child link="${name}_plate_link"/>
     </joint>

File: vito_description/robots/vito.urdf.xacro (robot description, xacro)
@@ -7,5 +7,6 @@
   <xacro:include filename="$(find lwr_description)/model/kuka_lwr.urdf.xacro"/>
   <xacro:include filename="$(find soft_hand_description)/model/soft_hand.urdf.xacro"/>
-  <link name="world_link" />
+  <xacro:include filename="$(find kit_head_description)/model/kit_head.urdf.xacro"/>
+  <link name="world" />
   <xacro:model_table name="table"
                     parent="world"
@@ -16,14 +17,23 @@
     <origin xyz="-1.22 0.5 0" rpy="0 0 0"/>
   </xacro:model_table>
-  <xacro:model_torso name="torso" parent="world_link">
+  <xacro:model_torso name="torso" parent="world">
     <origin xyz="0 0 0"/>
   </xacro:model_torso>
-  <xacro:kuka_lwr parent="world_link" name="left">
+  <xacro:kuka_lwr name="left" parent="world">
     <origin xyz="0.0 -0.108585 0.475"
       rpy="${M_PI*40.8933907/180} ${M_PI*48.5903708/180} ${M_PI*-40.8933907/180}"/>
   </xacro:kuka_lwr>
-  <xacro:kuka_lwr parent="world_link" name="right">
+  <xacro:kuka_lwr name="right" parent="world">
     <origin xyz="0.0 0.108585 0.475"
       rpy="${M_PI*-40.8933907/180} ${M_PI*48.5903708/180} ${M_PI*40.8933907/180}"/>
   </xacro:kuka_lwr>
+  <xacro:soft_hand parent="left_arm_7_link" name="left_hand" withAdaptiveTransmission="true" useMimicTag="$(arg use_mimic_tag)">
+    <origin xyz="0 0 0" rpy="1.570796 0 0"/>
+  </xacro:soft_hand>
+  <xacro:soft_hand parent="right_arm_7_link" name="right_hand" withAdaptiveTransmission="true" useMimicTag="$(arg use_mimic_tag)">
+    <origin xyz="0 0 0" rpy="1.570796 0 0"/>
+  </xacro:soft_hand>
+  <xacro:kit_head name="head" parent="world">
+    <origin xyz="0.0 0.0 ${0.55 + 0.1}" rpy="0.0 0.0 3.141592"/>
+  </xacro:kit_head>
 </robot>

Commit message: update on vito description

File: vito_description/model/table.urdf.xacro (robot description, xacro)
@@ -3,4 +3,16 @@
 <xacro:property name="leg_width" value="0.03" />
 <xacro:property name="border_offset" value="0.055" />
+<!-- conversions -->
+<!-- I couldn't make the simulation work with realistic values, so I tweaked the conversion values -->
+<xacro:property name="mm_to_m" value="0.001"/>
+<xacro:property name="mm2_to_m2" value="0.001"/>
+<xacro:property name="gr_to_Kg" value="0.01"/>
+<!-- not so negligible, otherwise simulation fails -->
+<xacro:property name="negligible_mass" value="${10*gr_to_Kg}"/>
+<xacro:property name="negligible_inertia">
+    <origin xyz="0 0 0"/>
+    <mass value="${negligible_mass}"/>
+    <inertia ixx="${negligible_mass * 10 * mm2_to_m2}" ixy="0.0" ixz="0.0" iyy="${negligible_mass * 10 * mm2_to_m2}" iyz="0.0" izz="${negligible_mass * 10 * mm2_to_m2}"/>
+</xacro:property>
 <xacro:macro name="table_leg" params="parent name *origin">
     <joint name="${name}_joint" type="fixed">
@@ -10,4 +22,7 @@
     </joint>
     <link name="${name}_link">
+        <inertial>
+            <insert_block name="negligible_inertia"/>
+        </inertial>
 		<visual>
 			<geometry>
@@ -22,4 +37,7 @@
 		</collision>
     </link>
+    <gazebo reference="${name}_link">
+        <static>true</static>
+    </gazebo>
 </xacro:macro>
 <xacro:macro name="model_table" params="parent name *origin length width height plate_thickness">
@@ -30,4 +48,7 @@
     </joint>
     <link name="${name}_plate_link">
+        <inertial>
+            <insert_block name="negligible_inertia"/>
+        </inertial>
         <visual>
             <origin xyz="${1/2 * length} ${-1/2 * width} ${-1/2 * plate_thickness}"/>
@@ -56,4 +77,7 @@
         <origin xyz="${length - border_offset} -${width - border_offset} -${1/2 * (plate_thickness + height)}"/>
     </xacro:table_leg>
+    <gazebo reference="${name}_plate_link">
+        <static>true</static>
+    </gazebo>
 </xacro:macro>
 </robot>

File: vito_description/model/torso.urdf.xacro (robot description, xacro)
@@ -1,4 +1,16 @@
 <?xml version="1.0"?>
 <robot xmlns:xacro="http://www.ros.org/wiki/xacro">
+<!-- conversions -->
+<!-- I couldn't make the simulation work with realistic values, so I tweaked the conversion values -->
+<xacro:property name="mm_to_m" value="0.001"/>
+<xacro:property name="mm2_to_m2" value="0.001"/>
+<xacro:property name="gr_to_Kg" value="0.01"/>
+<!-- not so negligible, otherwise simulation fails -->
+<xacro:property name="negligible_mass" value="${10*gr_to_Kg}"/>
+<xacro:property name="negligible_inertia">
+    <origin xyz="0 0 0"/>
+    <mass value="${negligible_mass}"/>
+    <inertia ixx="${negligible_mass * 10 * mm2_to_m2}" ixy="0.0" ixz="0.0" iyy="${negligible_mass * 10 * mm2_to_m2}" iyz="0.0" izz="${negligible_mass * 10 * mm2_to_m2}"/>
+</xacro:property>
 <xacro:macro name="model_torso" params="parent name *origin">
   <joint name="${parent}_${name}_base_joint" type="fixed">
@@ -8,4 +20,7 @@
   </joint>
   <link name="${name}_link">
+    <inertial>
+      <insert_block name="negligible_inertia"/>
+    </inertial>
     <visual>
       <geometry>
@@ -20,4 +35,7 @@
     </collision>
   </link>
+  <gazebo reference="${name}_link">
+    <static>true</static>
+  </gazebo>
 </xacro:macro>
 </robot>

File: vito_description/robot/vito.urdf.xacro (robot description, xacro)
@@ -12,8 +12,8 @@
                     parent="world"
                     length="1.45"
-                    width="1"
+                    width="1.45"
                     height="0.9"
                     plate_thickness="0.1">
-    <origin xyz="-1.22 0.5 0" rpy="0 0 0"/>
+    <origin xyz="-1.22 0.75 0" rpy="0 0 0"/>
   </xacro:model_table>
   <xacro:model_torso name="torso" parent="world">
@@ -28,8 +28,8 @@
       rpy="${M_PI*-40.8933907/180} ${M_PI*48.5903708/180} ${M_PI*40.8933907/180}"/>
   </xacro:kuka_lwr>
-  <xacro:soft_hand parent="left_arm_7_link" name="left_hand" left="true" withAdaptiveTransmission="true" useMimicTag="false">
+  <xacro:soft_hand parent="left_arm_7_link" name="left_hand" left="true" withAdaptiveTransmission="true" useMimicTag="true">
     <origin xyz="0 0 0" rpy="0 0 0"/>
   </xacro:soft_hand>
-  <xacro:soft_hand parent="right_arm_7_link" name="right_hand" left="false" withAdaptiveTransmission="true" useMimicTag="false">
+  <xacro:soft_hand parent="right_arm_7_link" name="right_hand" left="false" withAdaptiveTransmission="true" useMimicTag="true">
     <origin xyz="0 0 0" rpy="0 0 0"/>
   </xacro:soft_hand>

Commit message: Table model updated.

File: vito_description/model/table.urdf.xacro (robot description, xacro)
@@ -1,5 +1,5 @@
 <?xml version="1.0"?>
 <robot xmlns:xacro="http://www.ros.org/wiki/xacro">
-<xacro:property name="leg_width" value="0.03" />
+<xacro:property name="leg_width" value="0.08" />
 <xacro:property name="border_offset" value="0.055" />
 <!-- conversions -->
@@ -27,5 +27,5 @@
 		<visual>
 			<geometry>
-				<box size="${leg_width} -${leg_width} ${height - plate_thickness}"/>
+				<box size="${leg_width/2} -${leg_width} ${height - plate_thickness}"/>
 			</geometry>
 			<material name="Vito/Black"/>
@@ -33,5 +33,5 @@
 		<collision>
 			<geometry>
-				<box size="${leg_width} -${leg_width} ${height - plate_thickness}"/>
+				<box size="${leg_width/2} -${leg_width} ${height - plate_thickness}"/>
 			</geometry>
 		</collision>
@@ -65,14 +65,14 @@
         </collision>
     </link>
-    <xacro:table_leg parent="${name}_plate_link" name="leg_0">
+    <xacro:table_leg parent="${name}_plate_link" name="${name}_leg_0">
         <origin xyz="${border_offset} -${border_offset} -${1/2 * (plate_thickness + height)}"/>
     </xacro:table_leg>
-    <xacro:table_leg parent="${name}_plate_link" name="leg_1">
+    <xacro:table_leg parent="${name}_plate_link" name="${name}_leg_1">
         <origin xyz="${length - border_offset} -${border_offset} -${1/2 * (plate_thickness + height)}"/>
     </xacro:table_leg>
-    <xacro:table_leg parent="${name}_plate_link" name="leg_2">
+    <xacro:table_leg parent="${name}_plate_link" name="${name}_leg_2">
         <origin xyz="${border_offset} -${width - border_offset} -${1/2 * (plate_thickness + height)}"/>
     </xacro:table_leg>
-    <xacro:table_leg parent="${name}_plate_link" name="leg_3">
+    <xacro:table_leg parent="${name}_plate_link" name="${name}_leg_3">
         <origin xyz="${length - border_offset} -${width - border_offset} -${1/2 * (plate_thickness + height)}"/>
     </xacro:table_leg>

Commit message: Giving more plausible values of table and torso mass/inertia.

File: vito_description/model/table.urdf.xacro (robot description, xacro)
@@ -6,12 +6,12 @@
 <!-- I couldn't make the simulation work with realistic values, so I tweaked the conversion values -->
 <xacro:property name="mm_to_m" value="0.001"/>
-<xacro:property name="mm2_to_m2" value="0.001"/>
-<xacro:property name="gr_to_Kg" value="0.01"/>
+<xacro:property name="mm2_to_m2" value="0.000001"/>
+<xacro:property name="gr_to_Kg" value="0.001"/>
 <!-- not so negligible, otherwise simulation fails -->
-<xacro:property name="negligible_mass" value="${10*gr_to_Kg}"/>
-<xacro:property name="negligible_inertia">
+<xacro:property name="table_mass" value="${40000*gr_to_Kg}"/>
+<xacro:property name="table_inertia">
     <origin xyz="0 0 0"/>
-    <mass value="${negligible_mass}"/>
-    <inertia ixx="${negligible_mass * 10 * mm2_to_m2}" ixy="0.0" ixz="0.0" iyy="${negligible_mass * 10 * mm2_to_m2}" iyz="0.0" izz="${negligible_mass * 10 * mm2_to_m2}"/>
+    <mass value="${table_mass}"/>
+    <inertia ixx="${table_mass * 10 * mm2_to_m2}" ixy="0.0" ixz="0.0" iyy="${table_mass * 10 * mm2_to_m2}" iyz="0.0" izz="${table_mass * 10 * mm2_to_m2}"/>
 </xacro:property>
 <xacro:macro name="table_leg" params="parent name *origin">
@@ -23,5 +23,5 @@
     <link name="${name}_link">
         <inertial>
-            <insert_block name="negligible_inertia"/>
+            <insert_block name="table_inertia"/>
         </inertial>
 		<visual>
@@ -49,5 +49,5 @@
     <link name="${name}_plate_link">
         <inertial>
-            <insert_block name="negligible_inertia"/>
+            <insert_block name="table_inertia"/>
         </inertial>
         <visual>

File: vito_description/model/torso.urdf.xacro (robot description, xacro)
@@ -4,12 +4,12 @@
 <!-- I couldn't make the simulation work with realistic values, so I tweaked the conversion values -->
 <xacro:property name="mm_to_m" value="0.001"/>
-<xacro:property name="mm2_to_m2" value="0.001"/>
-<xacro:property name="gr_to_Kg" value="0.01"/>
+<xacro:property name="mm2_to_m2" value="0.000001"/>
+<xacro:property name="gr_to_Kg" value="0.001"/>
 <!-- not so negligible, otherwise simulation fails -->
-<xacro:property name="negligible_mass" value="${10*gr_to_Kg}"/>
-<xacro:property name="negligible_inertia">
+<xacro:property name="torso_mass" value="${20000*gr_to_Kg}"/>
+<xacro:property name="torso_inertia">
     <origin xyz="0 0 0"/>
-    <mass value="${negligible_mass}"/>
-    <inertia ixx="${negligible_mass * 10 * mm2_to_m2}" ixy="0.0" ixz="0.0" iyy="${negligible_mass * 10 * mm2_to_m2}" iyz="0.0" izz="${negligible_mass * 10 * mm2_to_m2}"/>
+    <mass value="${torso_mass}"/>
+    <inertia ixx="${torso_mass * 10 * mm2_to_m2}" ixy="0.0" ixz="0.0" iyy="${torso_mass * 10 * mm2_to_m2}" iyz="0.0" izz="${torso_mass * 10 * mm2_to_m2}"/>
 </xacro:property>
 <xacro:macro name="model_torso" params="parent name *origin">
@@ -21,5 +21,5 @@
   <link name="${name}_link">
     <inertial>
-      <insert_block name="negligible_inertia"/>
+      <insert_block name="torso_inertia"/>
     </inertial>
     <visual>

Commit message: trying to fix masses issues

File: vito_description/model/table.urdf.xacro (robot description, xacro)
@@ -9,9 +9,9 @@
 <xacro:property name="gr_to_Kg" value="0.001"/>
 <!-- not so negligible, otherwise simulation fails -->
-<xacro:property name="table_mass" value="${40000*gr_to_Kg}"/>
+<xacro:property name="table_mass" value="${40000*0.001}"/>
 <xacro:property name="table_inertia">
     <origin xyz="0 0 0"/>
     <mass value="${table_mass}"/>
-    <inertia ixx="${table_mass * 10 * mm2_to_m2}" ixy="0.0" ixz="0.0" iyy="${table_mass * 10 * mm2_to_m2}" iyz="0.0" izz="${table_mass * 10 * mm2_to_m2}"/>
+    <inertia ixx="${40 * 10 * 0.000001}" ixy="0.0" ixz="0.0" iyy="${40 * 10 * 0.000001}" iyz="0.0" izz="${40 * 10 * 0.000001}"/>
 </xacro:property>
 <xacro:macro name="table_leg" params="parent name *origin">

File: vito_description/model/torso.urdf.xacro (robot description, xacro)
@@ -7,9 +7,9 @@
 <xacro:property name="gr_to_Kg" value="0.001"/>
 <!-- not so negligible, otherwise simulation fails -->
-<xacro:property name="torso_mass" value="${20000*gr_to_Kg}"/>
+<xacro:property name="torso_mass" value="${20000*0.001}"/>
 <xacro:property name="torso_inertia">
     <origin xyz="0 0 0"/>
     <mass value="${torso_mass}"/>
-    <inertia ixx="${torso_mass * 10 * mm2_to_m2}" ixy="0.0" ixz="0.0" iyy="${torso_mass * 10 * mm2_to_m2}" iyz="0.0" izz="${torso_mass * 10 * mm2_to_m2}"/>
+    <inertia ixx="${20 * 10 * 0.000001}" ixy="0.0" ixz="0.0" iyy="${20 * 10 * 0.000001}" iyz="0.0" izz="${20 * 10 * 0.000001}"/>
 </xacro:property>
 <xacro:macro name="model_torso" params="parent name *origin">

File: vito_description/robot/vito.urdf.xacro (robot description, xacro)
@@ -9,6 +9,6 @@
   <xacro:include filename="$(find soft_hand_description)/model/soft_hand.urdf.xacro"/>
   <link name="world" />
-  <link name="vito_anchor" />
-    <joint name="w_fixed" type="fixed">
+   <link name="vito_anchor"/>
+  <joint name="w_fixed" type="fixed">
       <origin xyz="0.0 0.0 0.0" rpy="0 0 0"/>
       <parent link="world" />
@@ -16,25 +16,25 @@
     </joint>
   <!-- BODY -->
-  <xacro:model_table name="table"
+<!--    <xacro:model_table name="table"
                     parent="vito_anchor"
                     length="0.725"
                     width="1.05"
                     height="0.910"
-                    plate_thickness="0.05">
+		       plate_thickness="0.05">
     <origin xyz="0.0 0.55 0" rpy="0 0 0"/>
-  </xacro:model_table>
+    </xacro:model_table> -->
   <!-- WORKBENCH -->
-  <xacro:model_table name="workbench"
-                    parent="vito_anchor"
-                    length="0.725"
-                    width="1.25"
-                    height="0.960"
-                    plate_thickness="0.1">
-  <origin xyz="-1.25 0.625 0.07" rpy="0 0 0"/>
-  </xacro:model_table>
+<!--   <xacro:model_table name="workbench" -->
+<!--                     parent="vito_anchor" -->
+<!--                     length="0.725" -->
+<!--                     width="1.25" -->
+<!--                     height="0.960" -->
+<!--                     plate_thickness="0.1"> -->
+<!--   <origin xyz="-1.25 0.625 0.07" rpy="0 0 0"/> -->
+<!--   </xacro:model_table> -->
   <!-- TORSO -->
-  <xacro:model_torso name="torso" parent="vito_anchor">
+   <xacro:model_torso name="torso" parent="vito_anchor"> -->
     <origin xyz="0 0 0"/>
-  </xacro:model_torso>
+   </xacro:model_torso>
   <!-- LEFT ARM -->
   <xacro:kuka_lwr name="left_arm" parent="vito_anchor">
