Commit message: Changes the peek configuration and adds room to avoid crazy planning

File: vito_description/robot/vito_exploration.urdf.xacro (robot description, xacro)
@@ -51,5 +51,45 @@
   <!-- HEAD -->
   <xacro:kit_head name="head" parent="vito_anchor">
-    <origin xyz="0.0 0.0 ${0.55 + 0.1}" rpy="0.0 0.0 3.141592"/>
+    <origin xyz="-0.1 0.0 ${0.55 + 0.1}" rpy="0.0 0.0 3.141592"/>
   </xacro:kit_head>
+  <!-- Obstacles to reduce the workspace -->
+  <joint name="box1_joint" type="fixed">
+    <origin xyz="0 0 0" rpy="0 0 0"/>
+    <parent link="vito_anchor"/>
+    <child link="box1"/>
+  </joint>
+  <link name="box1">
+    <collision>
+      <origin xyz="0.0 0.0 0.0" rpy="0 0 0"/>
+      <geometry>
+        <box size="0.25 3.0 3.0"/>
+      </geometry>
+    </collision>
+  </link>
+  <joint name="box2_joint" type="fixed">
+    <origin xyz="0 1.1 0" rpy="0 0 1.57"/>
+    <parent link="vito_anchor"/>
+    <child link="box2"/>
+  </joint>
+  <link name="box2">
+    <collision>
+      <origin xyz="0.0 0.0 0.0" rpy="0 0 0"/>
+      <geometry>
+        <box size="0.1 3.0 3.0"/>
+      </geometry>
+    </collision>
+  </link>
+  <joint name="box3_joint" type="fixed">
+    <origin xyz="0 -1.1 0" rpy="0 0 1.57"/>
+    <parent link="vito_anchor"/>
+    <child link="box3"/>
+  </joint>
+  <link name="box3">
+    <collision>
+      <origin xyz="0.0 0.0 0.0" rpy="0 0 0"/>
+      <geometry>
+        <box size="0.1 3.0 3.0"/>
+      </geometry>
+    </collision>
+  </link>
 </robot>

Commit message: Adds walls to avoid crazy motions
No time to indague on a better moveit configuration.

Proper collision checking are disable for such end.

File: vito_description/robot/vito_exploration.urdf.xacro (robot description, xacro)
@@ -55,5 +55,5 @@
   <!-- Obstacles to reduce the workspace -->
   <joint name="box1_joint" type="fixed">
-    <origin xyz="0 0 0" rpy="0 0 0"/>
+    <origin xyz="-0.1 0 0" rpy="0 0 0"/>
     <parent link="vito_anchor"/>
     <child link="box1"/>
@@ -93,3 +93,45 @@
     </collision>
   </link>
+  <!-- front box -->
+  <joint name="box4left1_joint" type="fixed">
+    <origin xyz="-0.5 0.15 0.25" rpy="0 0 0"/>
+    <parent link="vito_anchor"/>
+    <child link="box4left1"/>
+  </joint>
+  <link name="box4left1">
+    <collision>
+      <origin xyz="0.0 0.0 0.0" rpy="0 0 0"/>
+      <geometry>
+        <box size="0.1 0.5 1.0"/>
+      </geometry>
+    </collision>
+  </link>
+  <!-- top box -->
+  <joint name="box4left2_joint" type="fixed">
+    <origin xyz="-0.9 0.15 0.75" rpy="0 0 0"/>
+    <parent link="vito_anchor"/>
+    <child link="box4left2"/>
+  </joint>
+  <link name="box4left2">
+    <collision>
+      <origin xyz="0.0 0.0 0.0" rpy="0 0 0"/>
+      <geometry>
+        <box size="0.8 0.8 0.1"/>
+      </geometry>
+    </collision>
+  </link>
+  <!-- bottom box -->
+  <joint name="box4left3_joint" type="fixed">
+    <origin xyz="-0.9 0.15 -0.25" rpy="0 0 0"/>
+    <parent link="vito_anchor"/>
+    <child link="box4left3"/>
+  </joint>
+  <link name="box4left3">
+    <collision>
+      <origin xyz="0.0 0.0 0.0" rpy="0 0 0"/>
+      <geometry>
+        <box size="0.8 0.8 0.1"/>
+      </geometry>
+    </collision>
+  </link>
 </robot>
