Commit message: add cutter to display_simple.urdf.xacro

File: vito_description/robot/vito_simple.urdf.xacro (robot description, xacro)
@@ -5,4 +5,5 @@
   <xacro:include filename="$(find vito_description)/model/materials.urdf"/>
   <xacro:include filename="$(find lwr_description)/model/kuka_lwr.urdf.xacro"/>
+  <xacro:include filename="$(find vito_description)/model/cutter.urdf.xacro"/>
   <link name="vito_anchor" />
   <!-- LEFT ARM -->
@@ -14,3 +15,7 @@
     <origin xyz="0.770 0.550 1.607" rpy="-2.428 -0.362 -1.183"/>
   </xacro:kuka_lwr>
+  <!-- CUTTER -->
+  <xacro:cutter parent="left_arm_7_link" name="cutter">
+    <origin xyz="0 0 0" rpy="0 0 0"/>
+  </xacro:cutter>
 </robot>

Commit message: add displacement between cutter and arm

File: vito_description/robot/vito_simple.urdf.xacro (robot description, xacro)
@@ -17,5 +17,5 @@
   <!-- CUTTER -->
   <xacro:cutter parent="left_arm_7_link" name="cutter">
-    <origin xyz="0 0 0" rpy="0 0 0"/>
+    <origin xyz="0 0 0.045" rpy="0 0 0"/>
   </xacro:cutter>
 </robot>

Commit message: added fixed joint between world and vito anchor not to have the robot fall

File: vito_description/robot/vito_simple.urdf.xacro (robot description, xacro)
@@ -6,5 +6,11 @@
   <xacro:include filename="$(find lwr_description)/model/kuka_lwr.urdf.xacro"/>
   <xacro:include filename="$(find vito_description)/model/cutter.urdf.xacro"/>
+  <link name="world" />
   <link name="vito_anchor" />
+  <joint name="w_fixed" type="fixed">
+    <origin xyz="0.0 0.0 0.0" rpy="0.0 0.0 0.0" />
+    <parent link="world" />
+    <child link="vito_anchor"/>
+  </joint>
   <!-- LEFT ARM -->
   <xacro:kuka_lwr name="left_arm" parent="vito_anchor">
