Commit message: Adding the qbmove-softhand clamp.

File: vito_description/robot/vito.urdf.xacro (robot description, xacro)
@@ -5,8 +5,10 @@
   <xacro:include filename="$(find vito_description)/model/table.urdf.xacro"/>
   <xacro:include filename="$(find vito_description)/model/materials.urdf"/>
+  <xacro:include filename="$(find vito_description)/model/clamp.urdf.xacro"/>
   <xacro:include filename="$(find lwr_description)/model/kuka_lwr.urdf.xacro"/>
   <xacro:include filename="$(find soft_hand_description)/model/soft_hand.urdf.xacro"/>
   <xacro:include filename="$(find kit_head_description)/model/kit_head.urdf.xacro"/>
   <link name="world" />
+  <!-- TABLE -->
   <xacro:model_table name="table"
                     parent="world"
@@ -17,21 +19,31 @@
     <origin xyz="-1.22 0.75 0" rpy="0 0 0"/>
   </xacro:model_table>
+  <!-- TORSO -->
   <xacro:model_torso name="torso" parent="world">
     <origin xyz="0 0 0"/>
   </xacro:model_torso>
+  <!-- LEFT ARM -->
   <xacro:kuka_lwr name="left_arm" parent="world">
     <origin xyz="0.0 -0.108585 0.475"
       rpy="${M_PI*40.8933907/180} ${M_PI*48.5903708/180} ${M_PI*-40.8933907/180}"/>
   </xacro:kuka_lwr>
+  <xacro:clamp name="left_clamp" parent="left_arm_7_link">
+    <origin xyz="0 0 0.01" rpy="0 0 0"/>
+  </xacro:clamp>
+  <xacro:soft_hand parent="left_clamp" name="left_hand" left="true" withAdaptiveTransmission="true" useMimicTag="false">
+    <origin xyz="0 0 0.004" rpy="0 0 0"/>
+  </xacro:soft_hand>
+  <!-- RIGHT ARM -->
   <xacro:kuka_lwr name="right_arm" parent="world">
     <origin xyz="0.0 0.108585 0.475"
       rpy="${M_PI*-40.8933907/180} ${M_PI*48.5903708/180} ${M_PI*40.8933907/180}"/>
   </xacro:kuka_lwr>
-  <xacro:soft_hand parent="left_arm_7_link" name="left_hand" left="true" withAdaptiveTransmission="true" useMimicTag="false">
-    <origin xyz="0 0 0" rpy="0 0 0"/>
+  <xacro:clamp name="right_clamp" parent="right_arm_7_link">
+    <origin xyz="0 0 0.01" rpy="0 0 0"/>
+  </xacro:clamp>
+  <xacro:soft_hand parent="right_clamp" name="right_hand" left="false" withAdaptiveTransmission="true" useMimicTag="false">
+    <origin xyz="0 0 0.004" rpy="0 0 0"/>
   </xacro:soft_hand>
-  <xacro:soft_hand parent="right_arm_7_link" name="right_hand" left="false" withAdaptiveTransmission="true" useMimicTag="false">
-    <origin xyz="0 0 0" rpy="0 0 0"/>
-  </xacro:soft_hand>
+  <!-- HEAD -->
   <xacro:kit_head name="head" parent="world">
     <origin xyz="0.0 0.0 ${0.55 + 0.1}" rpy="0.0 0.0 3.141592"/>

Commit message: Added the pacman version of the hand with couplers. @hamalMarino @alessandrosettimi @MirkoFerrati simulation will not work with this commit until CentroEPiaggio/pisa-iit-soft-hand#3 and CentroEPiaggio/kuka-lwr#3 are closed, which will be the default setup of Vito

File: vito_description/robot/vito.urdf.xacro (robot description, xacro)
@@ -6,6 +6,4 @@
   <xacro:include filename="$(find vito_description)/model/table.urdf.xacro"/>
   <xacro:include filename="$(find vito_description)/model/materials.urdf"/>
-  <xacro:include filename="$(find vito_description)/model/clamp.urdf.xacro"/>
-  <xacro:include filename="$(find vito_description)/model/softhand_base.urdf.xacro"/>
   <xacro:include filename="$(find lwr_description)/model/kuka_lwr.urdf.xacro"/>
   <xacro:include filename="$(find soft_hand_description)/model/soft_hand.urdf.xacro"/>
@@ -30,14 +28,7 @@
       rpy="${M_PI*40.8933907/180} ${M_PI*48.5903708/180} ${M_PI*-40.8933907/180}"/>
   </xacro:kuka_lwr>
-  <!-- LEFT COUPLERS -->
-  <xacro:clamp name="left_clamp" parent="left_arm_7_link">
-    <origin xyz="0 0 0.01" rpy="0 0 0"/>
-  </xacro:clamp>
-  <xacro:softhand_base name="left_base" parent="left_clamp" left="true">
-    <origin xyz="0 0 0.004" rpy="0 0 0"/>
-  </xacro:softhand_base>
   <!-- LEFT SOFTHAND -->
-  <xacro:soft_hand parent="left_base" name="left_hand" left="true" withAdaptiveTransmission="true" useMimicTag="true">
-    <origin xyz="0 0 0.0535" rpy="0 0 0"/>
+  <xacro:soft_hand parent="left_arm_7_link" name="left_hand" left="true" withAdaptiveTransmission="true" useMimicTag="true">
+    <origin xyz="0 0 0" rpy="0 0 0"/>
   </xacro:soft_hand>
   <!-- RIGHT ARM -->
@@ -46,14 +37,7 @@
       rpy="${M_PI*-40.8933907/180} ${M_PI*48.5903708/180} ${M_PI*40.8933907/180}"/>
   </xacro:kuka_lwr>
-  <!-- RIGHT COUPLERS -->
-  <xacro:clamp name="right_clamp" parent="right_arm_7_link">
-    <origin xyz="0 0 0.01" rpy="0 0 0"/>
-  </xacro:clamp>
-  <xacro:softhand_base name="right_base" parent="right_clamp" left="false">
-    <origin xyz="0 0 0.004" rpy="0 0 0"/>
-  </xacro:softhand_base>
   <!-- RIGHT SOFTHAND -->
-  <xacro:soft_hand parent="right_base" name="right_hand" left="false" withAdaptiveTransmission="true" useMimicTag="true">
-    <origin xyz="0 0 0.0535" rpy="0 0 0"/>
+  <xacro:soft_hand parent="right_arm_7_link" name="right_hand" left="false" withAdaptiveTransmission="true" useMimicTag="true">
+    <origin xyz="0 0 0" rpy="0 0 0"/>
   </xacro:soft_hand>
   <!-- HEAD -->

Commit message: [vito_description] Box added to compensate the table error.

File: vito_description/robot/vito.urdf.xacro (robot description, xacro)
@@ -45,3 +45,23 @@
     <origin xyz="0.0 0.0 ${0.55 + 0.1}" rpy="0.0 0.0 3.141592"/>
   </xacro:kit_head>
+  <!-- TEMPORAL BOX, DO NOT COMMIT IT! -->
+  <joint name="box_world_joint" type="fixed">
+        <origin xyz="-1.22 0.75 0.055" rpy="0 0 0"/>
+        <parent link="world"/>
+        <child link="box"/>
+    </joint>
+    <link name="box">
+        <visual>
+            <origin xyz="${1/2 * 1.45} ${-1/2 * 1.45} ${-1/2 * 0.055}"/>
+            <geometry>
+                <box size="1.45 1.45 0.055"/>
+      </geometry>
+    </visual>
+        <collision>
+            <origin xyz="${1/2 * 1.45} ${-1/2 * 1.45} ${-1/2 * 0.055}"/>
+            <geometry>
+                <box size="1.45 1.45 0.055"/>
+            </geometry>
+        </collision>
+    </link>
 </robot>

Commit message: Deleting the temporal box used to reproduce the high of the workbench.

File: vito_description/robot/vito.urdf.xacro (robot description, xacro)
@@ -45,23 +45,3 @@
     <origin xyz="0.0 0.0 ${0.55 + 0.1}" rpy="0.0 0.0 3.141592"/>
   </xacro:kit_head>
-  <!-- TEMPORAL BOX, DO NOT COMMIT IT! -->
-  <joint name="box_world_joint" type="fixed">
-        <origin xyz="-1.22 0.75 0.055" rpy="0 0 0"/>
-        <parent link="world"/>
-        <child link="box"/>
-    </joint>
-    <link name="box">
-        <visual>
-            <origin xyz="${1/2 * 1.45} ${-1/2 * 1.45} ${-1/2 * 0.055}"/>
-            <geometry>
-                <box size="1.45 1.45 0.055"/>
-      </geometry>
-    </visual>
-        <collision>
-            <origin xyz="${1/2 * 1.45} ${-1/2 * 1.45} ${-1/2 * 0.055}"/>
-            <geometry>
-                <box size="1.45 1.45 0.055"/>
-            </geometry>
-        </collision>
-    </link>
 </robot>

Commit message: The environment is set in environment.urdf.xacro that is spawned to Gazebo. Moveit sees the environment using Octomap. There is a template to load an environment when only kinematic planning is used in environment.yaml/display.launch. The .srdf has been updated to reflect that the robot now floats in Gazebo. Also the RVIZ configuration has been updated. This closes CentroEPiaggio/pacman-DR53#1

File: vito_description/robot/vito.urdf.xacro (robot description, xacro)
@@ -9,20 +9,20 @@
   <xacro:include filename="$(find soft_hand_description)/model/soft_hand.urdf.xacro"/>
   <xacro:include filename="$(find kit_head_description)/model/kit_head.urdf.xacro"/>
-  <link name="world" />
-  <!-- TABLE -->
+  <link name="vito_anchor" />
+  <!-- BODY -->
   <xacro:model_table name="table"
-                    parent="world"
-                    length="1.45"
-                    width="1.45"
-                    height="0.9"
-                    plate_thickness="0.1">
-    <origin xyz="-1.22 0.75 0" rpy="0 0 0"/>
+                    parent="vito_anchor"
+                    length="0.725"
+                    width="1.05"
+                    height="0.910"
+                    plate_thickness="0.05">
+    <origin xyz="-0.495 0.55 0" rpy="0 0 0"/>
   </xacro:model_table>
   <!-- TORSO -->
-  <xacro:model_torso name="torso" parent="world">
+  <xacro:model_torso name="torso" parent="vito_anchor">
     <origin xyz="0 0 0"/>
   </xacro:model_torso>
   <!-- LEFT ARM -->
-  <xacro:kuka_lwr name="left_arm" parent="world">
+  <xacro:kuka_lwr name="left_arm" parent="vito_anchor">
     <origin xyz="0.0 -0.108585 0.475"
       rpy="${M_PI*40.8933907/180} ${M_PI*48.5903708/180} ${M_PI*-40.8933907/180}"/>
@@ -33,5 +33,5 @@
   </xacro:soft_hand>
   <!-- RIGHT ARM -->
-  <xacro:kuka_lwr name="right_arm" parent="world">
+  <xacro:kuka_lwr name="right_arm" parent="vito_anchor">
     <origin xyz="0.0 0.108585 0.475"
       rpy="${M_PI*-40.8933907/180} ${M_PI*48.5903708/180} ${M_PI*40.8933907/180}"/>
@@ -42,5 +42,5 @@
   </xacro:soft_hand>
   <!-- HEAD -->
-  <xacro:kit_head name="head" parent="world">
+  <xacro:kit_head name="head" parent="vito_anchor">
     <origin xyz="0.0 0.0 ${0.55 + 0.1}" rpy="0.0 0.0 3.141592"/>
   </xacro:kit_head>

Commit message: Octomap is out, now vito includes the workbench as well /cc @hamalMarino You can use this version of vito, let me know if you find troubles.

File: vito_description/robot/vito.urdf.xacro (robot description, xacro)
@@ -18,4 +18,13 @@
                     plate_thickness="0.05">
     <origin xyz="-0.495 0.55 0" rpy="0 0 0"/>
+  </xacro:model_table>
+  <!-- WORKBENCH -->
+  <xacro:model_table name="workbench"
+                    parent="vito_anchor"
+                    length="0.725"
+                    width="1.05"
+                    height="0.960"
+                    plate_thickness="0.1">
+  <origin xyz="-1.25 0.55 0.05" rpy="0 0 0"/>
   </xacro:model_table>
   <!-- TORSO -->

Commit message: VITO READY TO WEAR A NICE SHIRT /cc @CentroEPiaggio/pacmandemoteam

File: vito_description/robot/vito.urdf.xacro (robot description, xacro)
@@ -34,6 +34,5 @@
   <!-- LEFT ARM -->
   <xacro:kuka_lwr name="left_arm" parent="vito_anchor">
-    <origin xyz="0.0 -0.108585 0.475"
-      rpy="${M_PI*40.8933907/180} ${M_PI*48.5903708/180} ${M_PI*-40.8933907/180}"/>
+    <origin xyz="-0.165 -0.1085854 0.390" rpy="1.5707963267948966 0.5235987010713441 -0.5235990737060282"/>
   </xacro:kuka_lwr>
   <!-- LEFT SOFTHAND -->
@@ -43,6 +42,5 @@
   <!-- RIGHT ARM -->
   <xacro:kuka_lwr name="right_arm" parent="vito_anchor">
-    <origin xyz="0.0 0.108585 0.475"
-      rpy="${M_PI*-40.8933907/180} ${M_PI*48.5903708/180} ${M_PI*40.8933907/180}"/>
+    <origin xyz="-0.165 0.10858 0.390" rpy="-1.5707963267948966 0.5235987010713441 0.5235990737060282"/>
   </xacro:kuka_lwr>
   <!-- RIGHT SOFTHAND -->

File: vito_description/robot/vito_calib.urdf.xacro (robot description, xacro)
@@ -30,10 +30,8 @@
   </xacro:model_torso>
   <xacro:kuka_lwr name="left_arm" parent="vito_anchor">
-    <origin xyz="0.0 -0.108585 0.475"
-      rpy="${M_PI*40.8933907/180} ${M_PI*48.5903708/180} ${M_PI*-40.8933907/180}"/>
+    <origin xyz="-0.165 -0.1085854 0.390" rpy="1.5707963267948966 0.5235987010713441 -0.5235990737060282"/>
   </xacro:kuka_lwr>
   <xacro:kuka_lwr name="right_arm" parent="vito_anchor">
-    <origin xyz="0.0 0.108585 0.475"
-      rpy="${M_PI*-40.8933907/180} ${M_PI*48.5903708/180} ${M_PI*40.8933907/180}"/>
+    <origin xyz="-0.165 0.10858 0.390" rpy="-1.5707963267948966 0.5235987010713441 0.5235990737060282"/>
   </xacro:kuka_lwr>
   <!-- from the CAD model, the frame coincides with the 7-th link -->

Commit message: Update on workbench geometry

File: vito_description/robot/vito.urdf.xacro (robot description, xacro)
@@ -26,5 +26,5 @@
                     height="0.960"
                     plate_thickness="0.1">
-  <origin xyz="-1.25 0.55 0.05" rpy="0 0 0"/>
+  <origin xyz="-1.25 0.55 0.07" rpy="0 0 0"/>
   </xacro:model_table>
   <!-- TORSO -->

Commit message: small tuning to robot model, home position and respawn

File: vito_description/robot/vito.urdf.xacro (robot description, xacro)
@@ -23,8 +23,8 @@
                     parent="vito_anchor"
                     length="0.725"
-                    width="1.05"
+                    width="1.25"
                     height="0.960"
                     plate_thickness="0.1">
-  <origin xyz="-1.25 0.55 0.07" rpy="0 0 0"/>
+  <origin xyz="-1.25 0.625 0.07" rpy="0 0 0"/>
   </xacro:model_table>
   <!-- TORSO -->

Commit message: updated vito-robot based on current real robot configuraiton

File: vito_description/robot/vito.urdf.xacro (robot description, xacro)
@@ -8,5 +8,5 @@
   <xacro:include filename="$(find lwr_description)/model/kuka_lwr.urdf.xacro"/>
   <xacro:include filename="$(find soft_hand_description)/model/soft_hand.urdf.xacro"/>
-  <xacro:include filename="$(find kit_head_description)/model/kit_head.urdf.xacro"/>
+  <!-- <xacro:include filename="$(find kit_head_description)/model/kit_head.urdf.xacro"/> -->
   <link name="vito_anchor" />
   <!-- BODY -->
@@ -42,5 +42,6 @@
   <!-- RIGHT ARM -->
   <xacro:kuka_lwr name="right_arm" parent="vito_anchor">
-    <origin xyz="-0.165 0.10858 0.390" rpy="-1.5707963267948966 0.5235987010713441 0.5235990737060282"/>
+    <!-- <origin xyz="-0.165 0.10858 0.390" rpy="-1.5707963267948966 0.5235987010713441 0.5235990737060282"/> -->
+    <origin xyz="-0.165 0.10858 0.390" rpy="-1.5707963267948966 -0.5235987010713441 0.5235990737060282"/>
   </xacro:kuka_lwr>
   <!-- RIGHT SOFTHAND -->
@@ -49,6 +50,6 @@
   </xacro:soft_hand>
   <!-- HEAD -->
-  <xacro:kit_head name="head" parent="vito_anchor">
+<!--   <xacro:kit_head name="head" parent="vito_anchor">
     <origin xyz="0.0 0.0 ${0.55 + 0.1}" rpy="0.0 0.0 3.141592"/>
-  </xacro:kit_head>
+  </xacro:kit_head> -->
 </robot>

Commit message: new commit

File: vito_description/robot/vito.urdf.xacro (robot description, xacro)
@@ -6,11 +6,69 @@
   <xacro:include filename="$(find vito_description)/model/table.urdf.xacro"/>
   <xacro:include filename="$(find vito_description)/model/materials.urdf"/>
-  <xacro:include filename="$(find lwr_description)/model/kuka_lwr.urdf.xacro"/>
+  <xacro:include filename="$(find lwr_description)/model/kuka_lwr_soma.urdf.xacro"/>
   <xacro:include filename="$(find soft_hand_description)/model/soft_hand.urdf.xacro"/>
   <!-- <xacro:include filename="$(find kit_head_description)/model/kit_head.urdf.xacro"/> -->
-  <link name="vito_anchor" />
+  <!-- CAM PARAMS FOR SOMA -->
+  <xacro:property name="cam_px" value="1.65" />
+  <xacro:property name="cam_py" value="-0.7" />
+  <xacro:property name="cam_pz" value="1.35" />
+  <xacro:property name="cam_or" value="-2.05" />
+  <xacro:property name="cam_op" value="0" />
+  <xacro:property name="cam_oy" value="0" />
+  <link name="world" />
+  <!-- KINECT FOR SOMA -->
+  <joint name="kinect2_rgb_joint" type="fixed">
+    <origin xyz="${cam_px} ${cam_py} ${cam_pz}" rpy="${cam_or} ${cam_op} ${cam_oy}"/>
+    <parent link="world"/>
+    <child link="kinect2_rgb_frame" />
+  </joint>
+  <link name="kinect2_rgb_frame"/>
+  <joint name="kinect2_joint" type="fixed">
+    <origin xyz="0.0 0.0 0.0" rpy="0 0 0"/>
+    <parent link="kinect2_rgb_frame"/>
+    <child link="kinect2_link"/>
+  </joint>
+  <link name="kinect2_link">
+    <visual>
+    <origin xyz="0 0 0" rpy="0 0 0"/>
+    <geometry>
+      <box size="0.05 0.05 0.05"/>
+    </geometry>
+    <material name="white">
+      <color rgba="1 1 0 1"/>
+    </material>
+    </visual>
+  </link>
+  <joint name="kinect2_rgb_optical_joint" type="fixed">
+    <origin xyz="0 0 0" rpy="0 0 0" />
+    <parent link="kinect2_link" />
+    <child link="kinect2_rgb_optical_frame" />
+  </joint>
+  <link name="kinect2_rgb_optical_frame"/>
+  <!-- THIS ONE MIGHT BE COMMENTED LATER -->
+  <joint name="kinect2_ir_optical_joint" type="fixed">
+    <origin xyz="0 0 0" rpy="0 0 0" />
+    <parent link="kinect2_rgb_optical_frame" />
+    <child link="kinect2_ir_optical_frame" />
+  </joint>
+  <link name="kinect2_ir_optical_frame"/>
+  <!-- THIS ONE MIGHT BE COMMENTED LATER -->
+  <!-- The fixed joints & links below are usually published by static_transformers launched by the iai _kinect files. However, for Gazebo simulation we need them, so we add them here. (Hence, don't publish them additionally!) -->
+  <joint name="kinect2_depth_joint" type="fixed">
+    <origin xyz="0 ${2 * -kinect_cam_py} 0" rpy="0 0 0" />
+    <parent link="kinect2_rgb_frame" />
+    <child link="kinect2_depth_frame" />
+  </joint>
+  <link name="kinect2_depth_frame"/>
+  <joint name="kinect2_depth_optical_joint" type="fixed">
+    <origin xyz="0 0 0" rpy="${_M_PI_2} 0 ${_M_PI_2}" />
+    <parent link="kinect2_depth_frame" />
+    <child link="kinect2_depth_optical_frame" />
+  </joint>
+  <link name="kinect2_depth_optical_frame"/>
+  <!-- Kinect Camera END -->
   <!-- BODY -->
-  <xacro:model_table name="table"
-                    parent="vito_anchor"
+<!--   <xacro:model_table name="table"
+                    parent="world"
                     length="0.725"
                     width="1.05"
@@ -18,8 +76,8 @@
                     plate_thickness="0.05">
     <origin xyz="-0.495 0.55 0" rpy="0 0 0"/>
-  </xacro:model_table>
+  </xacro:model_table> -->
   <!-- WORKBENCH -->
-  <xacro:model_table name="workbench"
-                    parent="vito_anchor"
+<!--   <xacro:model_table name="workbench"
+                    parent="world"
                     length="0.725"
                     width="1.25"
@@ -27,28 +85,29 @@
                     plate_thickness="0.1">
   <origin xyz="-1.25 0.625 0.07" rpy="0 0 0"/>
-  </xacro:model_table>
+  </xacro:model_table> -->
   <!-- TORSO -->
-  <xacro:model_torso name="torso" parent="vito_anchor">
+<!--   <xacro:model_torso name="torso" parent="world">
     <origin xyz="0 0 0"/>
-  </xacro:model_torso>
+  </xacro:model_torso> -->
   <!-- LEFT ARM -->
-  <xacro:kuka_lwr name="left_arm" parent="vito_anchor">
+  <!-- <xacro:kuka_lwr name="left_arm" parent="world">
     <origin xyz="-0.165 -0.1085854 0.390" rpy="1.5707963267948966 0.5235987010713441 -0.5235990737060282"/>
-  </xacro:kuka_lwr>
+    <origin xyz="0.57 0.801 1.307" rpy="3.1415 0.5235987010713441 3.1415"/>
+  </xacro:kuka_lwr>-->
   <!-- LEFT SOFTHAND -->
-  <xacro:soft_hand parent="left_arm_7_link" name="left_hand" left="true" withAdaptiveTransmission="true" useMimicTag="$(arg use_mimic_tag)">
-    <origin xyz="0 0 0" rpy="0 0 0"/>
-  </xacro:soft_hand>
+  <!-- <xacro:soft_hand parent="left_arm_7_link" name="left_hand" left="true" withAdaptiveTransmission="true" useMimicTag="$(arg use_mimic_tag)">
+    <origin xyz="0 0 0" rpy="0 0 0.5235987010713441"/>
+  </xacro:soft_hand> -->
   <!-- RIGHT ARM -->
-  <xacro:kuka_lwr name="right_arm" parent="vito_anchor">
+  <xacro:kuka_lwr name="right_arm" parent="world">
     <!-- <origin xyz="-0.165 0.10858 0.390" rpy="-1.5707963267948966 0.5235987010713441 0.5235990737060282"/> -->
-    <origin xyz="-0.165 0.10858 0.390" rpy="-1.5707963267948966 -0.5235987010713441 0.5235990737060282"/>
+ <origin xyz="0.77 0.801 1.607" rpy="3.1415 -0.7854 0"/>
   </xacro:kuka_lwr>
   <!-- RIGHT SOFTHAND -->
-  <xacro:soft_hand parent="right_arm_7_link" name="right_hand" left="false" withAdaptiveTransmission="true" useMimicTag="$(arg use_mimic_tag)">
-    <origin xyz="0 0 0" rpy="0 0 0"/>
+  <xacro:soft_hand parent="right_arm_link_ee" name="right_hand" left="false" withAdaptiveTransmission="true" useMimicTag="$(arg use_mimic_tag)">
+    <origin xyz="0 0 0" rpy="0 -1.5708 3.1415"/>
   </xacro:soft_hand>
   <!-- HEAD -->
-<!--   <xacro:kit_head name="head" parent="vito_anchor">
+<!--   <xacro:kit_head name="head" parent="world">
     <origin xyz="0.0 0.0 ${0.55 + 0.1}" rpy="0.0 0.0 3.141592"/>
   </xacro:kit_head> -->

Commit message: Working on cartesian impedance controller for reactive grasp

File: vito_description/robot/vito.urdf.xacro (robot description, xacro)
@@ -47,5 +47,5 @@
   <!-- RIGHT SOFTHAND -->
   <xacro:soft_hand parent="right_arm_7_link" name="right_hand" left="false" withAdaptiveTransmission="true" useMimicTag="$(arg use_mimic_tag)">
-    <origin xyz="0 0 0" rpy="0 0 0"/>
+    <origin xyz="0 1 0" rpy="0 0 0"/>
   </xacro:soft_hand>
   <!-- HEAD -->

File: vito_description/robot/vito_iliad.urdf.xacro (robot description, xacro)
@@ -153,5 +153,5 @@
       <disableFixedJointLumping>true</disableFixedJointLumping>
     </gazebo>  -->
-    <xacro:model_table name="table"
+    <!-- <xacro:model_table name="table"
                     parent="world"
                     length="0.6"
@@ -160,4 +160,4 @@
                     plate_thickness="0.05">
     <origin xyz="1.350 1.201 0.70" rpy="0 0 0"/>
-</xacro:model_table>
+</xacro:model_table> -->
 </robot>
